File: EZ-VIK/EZ-VIK.kicad_sch (KiCad schematic)
At the start: 4 parts, among them J2 Conn_01x04

Commit message: Split into full size and mini
Added Mini branch, and changed main branch to the full size VIK connector.
Parts:
- J4: footprint vik:vik-keyboard-connector-horizontal-mini -> vik:vik-keyboard-connector-horizontal
Changed lines of the file:
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@@
       (effects (font (size 1.27 1.27)))
     )
-    (property "Footprint" "vik:vik-keyboard-connector-horizontal-mini" (at 115.57 53.34 0)
+    (property "Footprint" "vik:vik-keyboard-connector-horizontal" (at 115.57 53.34 0)
       (effects (font (size 1.27 1.27)) hide)
     )
